Commit message: commit 2

File: camera/realsense2_description/urdf/_d435.gazebo.xacro (robot description, xacro)
@@ -13,5 +13,5 @@
       <enable_wind>0</enable_wind>
       <kinematic>0</kinematic>
-      <gravity>1</gravity>
+      <gravity>true</gravity>
       <!--<mu>1</mu>-->
       <mu2>1</mu2>

File: camera/realsense2_description/urdf/_t265.gazebo.xacro (robot description, xacro)
@@ -12,5 +12,5 @@
       <enable_wind>0</enable_wind>
       <kinematic>0</kinematic>
-      <gravity>1</gravity>
+      <gravity>true</gravity>
       <!--<mu>1</mu>-->
       <mu2>1</mu2>
@@ -79,5 +79,5 @@
       <enable_wind>0</enable_wind>
       <kinematic>0</kinematic>
-      <gravity>1</gravity>
+      <gravity>true</gravity>
       <!--<mu>1</mu>-->
       <mu2>1</mu2>

File: robot2/robot2_description/config/macro.gripper_assembly.xacro (robot description, xacro)
@@ -22,4 +22,8 @@
       </collision>
     </link>
+    <gazebo reference="gripper_mount_link">
+      <!-- <material>Gazebo/Grey</material> -->
+      <material>PR2/Grey3</material>
+    </gazebo>
     <!-- yf: Define gripper_mount_ud link -->
     <link name="gripper_mount_ud_link">
@@ -42,4 +46,7 @@
       </collision>
     </link>
+    <gazebo reference="gripper_mount_ud_link">
+      <material>Gazebo/Grey</material>
+    </gazebo>
     <!-- yf: Define gripper_L link -->
     <!-- <link name="gripper_L_link">

File: robot2/robot2_description/config/macro.top_module.xacro (robot description, xacro)
@@ -22,4 +22,7 @@
       </collision>
     </link>
+    <gazebo reference="top_module_link">
+      <material>Gazebo/Grey</material>
+    </gazebo>
   </xacro:macro>
 </robot>

File: robot2/robot2_description/urdf/robot2_v1.urdf.xacro (robot description, xacro)
@@ -42,4 +42,10 @@
       <dynamics damping="20000.0"/> -->
     </joint>
+    <!-- <transmission name="ud_gripper_mount_trans" type="robot2/SimpleTransmission">
+      <actuator name="ud_gripper_mount_motor"/>
+      <joint name="ud_gripper_mount_joint"/>
+      <mechanicalReduction>-47641.53</mechanicalReduction>
+      <simulated_actuated_joint name="torso_lift_motor_screw_joint" simulated_reduction="3141.6"/>
+    </transmission> -->
     <!-- <joint name="ud_gripper_mount_joint" type="fixed">
       <parent link="gripper_mount_link" />
