Commit message: commit 2.5

File: robot2/robot2_description/urdf/robot2.gazebo.xacro (robot description, xacro)
@@ -3,4 +3,33 @@
   <xacro:arg name="laser_visual" default="false"/>
   <xacro:arg name="imu_visual"   default="false"/>
+  <gazebo reference="caster1">
+    <mu1>0.1</mu1>
+    <mu2>0.1</mu2>
+    <kp>1000000.0</kp>
+    <kd>100.0</kd>
+    <minDepth>0.001</minDepth>
+    <maxVel>1.0</maxVel>
+    <material>Gazebo/FlatBlack</material>
+  </gazebo>
+  <!-- <gazebo reference="left_wheel">
+    <mu1>0.1</mu1>
+    <mu2>0.1</mu2>
+    <kp>500000.0</kp>
+    <kd>10.0</kd>
+    <minDepth>0.001</minDepth>
+    <maxVel>0.1</maxVel>
+    <fdir1>1 0 0</fdir1>
+    <material>Gazebo/FlatBlack</material>
+  </gazebo>
+  <gazebo reference="right_wheel">
+    <mu1>0.1</mu1>
+    <mu2>0.1</mu2>
+    <kp>500000.0</kp>
+    <kd>10.0</kd>
+    <minDepth>0.001</minDepth>
+    <maxVel>0.1</maxVel>
+    <fdir1>1 0 0</fdir1>
+    <material>Gazebo/FlatBlack</material>
+  </gazebo> -->
   <gazebo>
     <plugin name="turtlebot3_burger_controller" filename="libgazebo_ros_diff_drive.so">
@@ -94,12 +123,3 @@
     </sensor>
   </gazebo>
-  <gazebo reference="caster1">
-    <mu1>0.1</mu1>
-    <mu2>0.1</mu2>
-    <kp>1000000.0</kp>
-    <kd>100.0</kd>
-    <minDepth>0.001</minDepth>
-    <maxVel>1.0</maxVel>
-    <material>Gazebo/FlatBlack</material>
-  </gazebo>
 </robot>

File: robot2/robot2_description/urdf/robot2.urdf.xacro (robot description, xacro)
@@ -1,217 +1,14 @@
 <?xml version='1.0'?>
 <robot name="robot2" xmlns:xacro="http://ros.org/wiki/xacro">
- <xacro:include filename="$(find robot2_description)/urdf/robot2.gazebo.xacro"/>
- <xacro:include filename="$(find robot2_description)/urdf/common_properties.xacro"/>
- <!-- Spawn camera -->
- <xacro:include filename="$(find realsense2_description)/urdf/test_d435_camera.urdf.xacro" />
- <!-- base_footpint setup -->
- <link name="base_footprint"/>
- <joint name="base_joint" type="fixed">
-    <parent link="base_footprint"/>
-    <child link="base_link"/>
-    <origin xyz="0.0 0.0 0.13" rpy="0 0 0"/>
- </joint>
- <!-- Base Link -->
- <link name="base_link">
-    <visual>
-      <origin xyz="0 0 0" rpy="0 0 3.14" />
-      <geometry>
-          <mesh filename="package://robot2_description/meshes/bases/robot2_board_2.stl" scale="1 1 1"/>
-      </geometry>
-    </visual>
-    <!-- Base collision, mass and inertia -->
-    <collision>
-      <origin xyz="0 0 0" rpy="0 0 3.14" />
-      <geometry>
-          <mesh filename="package://robot2_description/meshes/bases/robot2_board_2.stl" scale="1 1 1"/>
-      </geometry>
-    </collision>
-    <inertial>
-      <mass value="5.0"/>
-      <inertia ixx="0.13" ixy="0.0" ixz="0.0" iyy="0.21" iyz="0.0" izz="0.13"/>
-    </inertial>
- </link>
-  <link name="caster1">
-   <visual>
-      <origin xyz="0 0 0" rpy="0 0 0" />
-      <geometry>
-        <sphere radius="0.065" />
-      </geometry>
-    </visual>
-    <!-- Caster1 collision, mass and inertia -->
-    <collision>
-      <origin xyz="0 0 0" rpy="0 0 0" />
-      <geometry>
-        <sphere radius="0.065" />
-      </geometry>
-    </collision>
-    <inertial>
-      <mass value="1.0"/>
-      <inertia ixx="0.00169" ixy="0.0" ixz="0.0" iyy="0.00169" iyz="0.0" izz="0.00169"/>
-    </inertial>
-  </link>
-  <joint name="caster_joint" type="fixed">
-    <parent link="base_link"/>
-    <child link="caster1"/>
-    <origin xyz="-0.2 0 -0.065" rpy="0 0 0"/>
-  </joint>
-  <!-- IMU  -->
-  <joint name="imu_joint" type="fixed">
-    <parent link="base_link"/>
-    <child link="imu_link"/>
-    <origin xyz="-0.032 0 0.068" rpy="0 0 0"/>
-  </joint>
-  <link name="imu_link"/>
-  <!-- Right Wheel -->
-  <link name="right_wheel">
-    <visual>
-      <origin xyz="0 0 0" rpy="1.570795 0 0" />
-      <geometry>
-          <cylinder length="0.05" radius="0.1"/>
-      </geometry>
-    </visual>
-    <!-- Right Wheel collision, mass and inertia -->
-    <collision>
-     <origin xyz="0 0 0" rpy="1.570795 0 0" />
-      <geometry>
-          <cylinder length="0.05" radius="0.1"/>
-      </geometry>
-    </collision>
-    <inertial>
-      <mass value="1.0"/>
-      <inertia ixx="0.01" ixy="0.0" ixz="0.0" iyy="0.005" iyz="0.0" izz="0.005"/>
-    </inertial>
-  </link>
-  <!-- Right Wheel joint -->
-  <joint name="joint_right_wheel" type="continuous">
-    <parent link="base_link"/>
-    <child link="right_wheel"/>
-    <origin xyz="0.2 -0.225 -0.030" rpy="0 0 0" />
-    <axis xyz="0 1 0" />
-  </joint>
-  <!-- Left Wheel -->
-  <link name="left_wheel">
-    <visual>
-      <origin xyz="0 0 0" rpy="1.570795 0 0" />
-      <geometry>
-          <cylinder length="0.05" radius="0.1"/>
-      </geometry>
-    </visual>
-    <!-- Left Wheel collision, mass and inertia -->
-    <collision>
-      <origin xyz="0 0 0" rpy="1.570795 0 0" />
-      <geometry>
-          <cylinder length="0.05" radius="0.1"/>
-      </geometry>
-    </collision>
-    <inertial>
-      <mass value="1.0"/>
-      <inertia ixx="0.01" ixy="0.0" ixz="0.0" iyy="0.005" iyz="0.0" izz="0.005"/>
-    </inertial>
-  </link>
-  <!-- Left Wheel joint -->
-  <joint name="joint_left_wheel" type="continuous">
-    <parent link="base_link"/>
-    <child link="left_wheel"/>
-    <origin xyz="0.2 0.225 -0.030" rpy="0 0 0"/>
-    <axis xyz="0 1 0"/>
-  </joint>
-  <!-- Lidar Stand-->
- <joint name="scan_stand_joint" type="fixed">
-    <parent link="base_link"/>
-    <child link="base_scan_stand"/>
-    <origin xyz="0.325 0 0.00" rpy="0 0 0"/>
-  </joint>
-  <link name="base_scan_stand">
-    <visual>
-      <origin xyz="0 0 0.0" rpy="0 0 0"/>
-      <geometry>
-          <box size="0.05 0.3 0.1" />
-       </geometry>
-     </visual>
-    <collision>
-      <origin xyz="0 0 0.0" rpy="0 0 0"/>
-      <geometry>
-          <box size="0.05 0.3 0.1" />
-      </geometry>
-    </collision>
-    <inertial>
-      <mass value="1.0" />
-      <origin xyz="0 0 0" />
-      <inertia ixx="0.001" ixy="0.0" ixz="0.0"
-               iyy="0.001" iyz="0.0"
-               izz="0.001" />
-    </inertial>
-  </link>
-<!-- back stand -->
-  <joint name="back_stand_joint" type="fixed">
-    <parent link="base_link"/>
-    <child link="back_stand"/>
-    <origin xyz="-0.275 0 0.085" rpy="0 0 0"/>
-  </joint>
-  <link name="back_stand">
-    <visual>
-      <origin xyz="0 0 0.0" rpy="0 0 0"/>
-      <geometry>
-          <box size="0.05 0.05 0.05" />
-       </geometry>
-     </visual>
-    <collision>
-      <origin xyz="0 0 0.0" rpy="0 0 0"/>
-      <geometry>
-          <box size="0.05 0.05 0.05" />
-      </geometry>
-    </collision>
-    <inertial>
-      <mass value="0.5" />
-      <origin xyz="0 0 0" />
-      <inertia ixx="0.001" ixy="0.0" ixz="0.0"
-               iyy="0.001" iyz="0.0"
-               izz="0.001" />
-    </inertial>
-  </link>
-  <!-- Lidar
-  <joint name="scan_joint" type="fixed">
-    <parent link="base_scan_stand"/>
-    <child link="base_scan"/>
-    <origin xyz="0 0 0.06" rpy="0 0 0"/>
-  </joint> -->
-  <!-- Lidar -->
-  <joint name="scan_joint" type="fixed">
-    <parent link="back_stand"/>
-    <child link="base_scan"/>
-    <origin xyz="0.0 0.0 0.0375" rpy="0 0 3.14"/>
-  </joint>
-  <link name="base_scan">
-    <visual>
-      <origin xyz="0 0 0.0" rpy="0 0 0"/>
-      <geometry>
-	 <cylinder length="0.030" radius="0.02"/>
-      </geometry>
-    </visual>
-    <collision>
-      <origin xyz="0 0 0.0" rpy="0 0 0"/>
-      <geometry>
-        <cylinder length="0.030" radius="0.02"/>
-      </geometry>
-    </collision>
-    <inertial>
-      <mass value="0.2" />
-      <origin xyz="0 0 0" />
-      <inertia ixx="0.001" ixy="0.0" ixz="0.0"
-               iyy="0.001" iyz="0.0"
-               izz="0.001" />
-    </inertial>
-  </link>
-<!--Attach camera to the top_module -->
-  <!-- <joint name="camera_top_module_joint" type="fixed">
-    <parent link="base_scan_stand" />
-    <child link="camera_base_link"/>
-    <origin xyz="0.02 0 0.00" rpy="0 0 0"/>
-  </joint> -->
-  <joint name="camera_top_module_joint" type="fixed">
-    <parent link="base_scan_stand" />
-    <child link="camera_base_link"/>
-    <origin xyz="0.01 0 0.05" rpy="0 0 0"/>
-  </joint>
+  <xacro:include filename="$(find robot2_description)/urdf/robot2_v1.urdf.xacro" />
+  <xacro:arg name="tf_prefix" default="" />
+  <xacro:property name="tf_prefix_" value="$(arg tf_prefix)" />
+  <xacro:if value="${tf_prefix_ == ''}">
+    <xacro:property name="prefix" value="" />
+  </xacro:if>
+  <xacro:unless value="${tf_prefix_ == ''}">
+    <xacro:property name="prefix" value="${tf_prefix_}/" />
+  </xacro:unless>
+  <xacro:robot2 prefix="${prefix}"/>
+  <!-- <xacro:controller_plugin_gazebo robot_namespace=""/> -->
 </robot>
